Commit message: feat: complete AMR simulation stack
- Modular URDF/Xacro: chassis, drive wheels, castors, lidar, gazebo plugins
- Gazebo Fortress simulation: custom world, URDF->SDF conversion, ROS bridge
- SLAM: slam_toolbox async mapping, map saved to maps/
- Nav2: AMCL localization, DWB planner, costmap, behavior tree navigation
- Launch files: display, gazebo, slam, nav2
- Known: double Gazebo instance and Nav2 behavior tree being debugged

File: my_amr_description/urdf/drive_wheels.xacro (robot description, xacro)
@@ -5,5 +5,5 @@
   <xacro:property name="traction_track_width"   value="0.36"/>
   <xacro:property name="chassis_height"         value="0.19"/>
-  <xacro:property name="trolley_wheel_radius"   value="0.04"/>
+  <xacro:property name="trolley_wheel_radius"   value="0.044"/>
   <xacro:property name="eps"                    value="0.002"/>
   <xacro:property name="wheel_mass"             value="1.5"/>
@@ -29,5 +29,5 @@
     <!-- exact bcr_bot formula for wheel z -->
     <joint name="${name}_joint" type="continuous">
-      <parent link="chassis_link"/>
+      <parent link="base_link"/>
       <child link="${name}_link"/>
       <origin xyz="0 ${y_reflect * traction_track_width/2} ${-(chassis_height/2 + 2*trolley_wheel_radius + eps - traction_wheel_radius)}" rpy="0 0 0"/>

File: my_amr_description/urdf/gazebo_control.xacro (robot description, xacro)
@@ -2,26 +2,23 @@
 <robot xmlns:xacro="http://www.ros.org/wiki/xacro">
   <gazebo>
-    <plugin name="diff_drive" filename="libgazebo_ros_diff_drive.so">
-      <ros>
-        <remapping>cmd_vel:=cmd_vel</remapping>
-        <remapping>odom:=odom</remapping>
-      </ros>
+    <plugin filename="libignition-gazebo6-diff-drive-system.so"
+            name="ignition::gazebo::systems::DiffDrive">
       <left_joint>left_wheel_joint</left_joint>
       <right_joint>right_wheel_joint</right_joint>
-      <!-- wheel_y_offset * 2 = 0.22 * 2 = 0.44 -->
       <wheel_separation>0.36</wheel_separation>
-      <!-- wheel_radius * 2 = 0.065 * 2 = 0.13 -->
-      <wheel_diameter>0.20</wheel_diameter>
+      <wheel_radius>0.10</wheel_radius>
       <max_wheel_torque>20</max_wheel_torque>
-      <max_wheel_acceleration>1.0</max_wheel_acceleration>
-      <publish_odom>true</publish_odom>
+      <max_wheel_acceleration>0.5</max_wheel_acceleration>
+      <topic>cmd_vel</topic>
+      <odom_topic>odom</odom_topic>
+      <frame_id>odom</frame_id>
+      <child_frame_id>base_footprint</child_frame_id>
       <publish_odom_tf>true</publish_odom_tf>
-      <publish_wheel_tf>true</publish_wheel_tf>
-      <odometry_frame>odom</odometry_frame>
-      <robot_base_frame>base_footprint</robot_base_frame>
+      <odom_publish_frequency>50</odom_publish_frequency>
     </plugin>
   </gazebo>
   <gazebo>
-    <plugin name="joint_state_publisher" filename="libgazebo_ros_joint_state_publisher.so">
+    <plugin filename="libignition-gazebo6-joint-state-publisher-system.so"
+            name="ignition::gazebo::systems::JointStatePublisher">
       <joint_name>left_wheel_joint</joint_name>
       <joint_name>right_wheel_joint</joint_name>

File: my_amr_description/urdf/lidar.xacro (robot description, xacro)
@@ -1,7 +1,4 @@
 <?xml version="1.0"?>
 <robot xmlns:xacro="http://www.ros.org/wiki/xacro">
-  <!-- ═══════════════════════════════════
-       LIDAR LINK
-  ═══════════════════════════════════ -->
   <link name="lidar_link">
     <visual>
@@ -18,20 +15,18 @@
     <xacro:cylinder_inertia m="0.2" r="0.05" h="0.07"/>
   </link>
-  <!-- fixed on top center of chassis -->
   <joint name="lidar_joint" type="fixed">
-    <parent link="base_link"/>
+    <parent link="chassis_link"/>
     <child link="lidar_link"/>
-    <origin xyz="0 0 0.085" rpy="0 0 0"/>
+    <origin xyz="0 0 0.13" rpy="0 0 0"/>
   </joint>
-  <!-- ═══════════════════════════════════
-       GAZEBO LIDAR SENSOR PLUGIN
-  ═══════════════════════════════════ -->
   <gazebo reference="lidar_link">
     <material>Gazebo/Grey</material>
-    <sensor name="lidar" type="ray">
+    <sensor name="lidar" type="gpu_lidar">
       <always_on>true</always_on>
       <visualize>true</visualize>
       <update_rate>10</update_rate>
-      <ray>
+      <topic>scan</topic>
+      <gz_frame_id>lidar_link</gz_frame_id>
+      <lidar>
         <scan>
           <horizontal>
@@ -39,10 +34,10 @@
             <resolution>1</resolution>
             <min_angle>-3.14159</min_angle>
-            <max_angle> 3.14159</max_angle>
+            <max_angle>3.14159</max_angle>
           </horizontal>
         </scan>
         <range>
           <min>0.12</min>
-          <max>20.0</max>
+          <max>16.0</max>
           <resolution>0.01</resolution>
         </range>
@@ -52,12 +47,5 @@
           <stddev>0.01</stddev>
         </noise>
-      </ray>
-      <plugin name="gazebo_ros_lidar" filename="libgazebo_ros_ray_sensor.so">
-        <ros>
-          <remapping>~/out:=scan</remapping>
-        </ros>
-        <output_type>sensor_msgs/LaserScan</output_type>
-        <frame_name>lidar_link</frame_name>
-      </plugin>
+      </lidar>
     </sensor>
   </gazebo>

File: my_amr_description/urdf/robot_base.xacro (robot description, xacro)
@@ -7,5 +7,5 @@
   <xacro:property name="chassis_mass"         value="12.0"/>
   <xacro:property name="traction_wheel_radius" value="0.10"/>
-  <xacro:property name="trolley_wheel_radius"  value="0.04"/>
+  <xacro:property name="trolley_wheel_radius"  value="0.044"/>
   <xacro:property name="trolley_track_width"   value="0.36"/>
   <xacro:property name="eps"                   value="0.002"/>
@@ -25,9 +25,9 @@
   <link name="base_footprint"/>
   <link name="base_link"/>
-  <!-- exact same formula as bcr_bot -->
+  <!-- z = chassis_height/2 + 2*trolley_wheel_radius + eps = 0.095 + 0.088 + 0.002 = 0.185 -->
   <joint name="base_footprint_joint" type="fixed">
     <parent link="base_footprint"/>
     <child link="base_link"/>
-    <origin xyz="0 0 ${chassis_height/2 + traction_wheel_radius}" rpy="0 0 0"/>
+    <origin xyz="0 0 0.185" rpy="0 0 0"/>
   </joint>
   <link name="chassis_link">

Commit message: Fix URDF errors, update map and launch files
- Fix lift_tray.xacro: move solid_black material to top level, fix gazebo reference tags
- Update robot_base.xacro and drive_wheels.xacro with corrected geometry
- Update gazebo_control.xacro with lift joint controller
- Add odom_tf_broadcaster.py: odometry TF broadcaster
- Update gazebo.launch.py with correct bridge topics
- Update CMakeLists.txt to install scripts
- Add generated warehouse map (my_map.pgm + my_map.yaml)

File: my_amr_description/urdf/drive_wheels.xacro (robot description, xacro)
@@ -7,5 +7,5 @@
   <xacro:property name="trolley_wheel_radius"   value="0.044"/>
   <xacro:property name="eps"                    value="0.002"/>
-  <xacro:property name="wheel_mass"             value="1.5"/>
+  <xacro:property name="wheel_mass"             value="30.0"/>
   <xacro:macro name="drive_wheel" params="name y_reflect">
     <link name="${name}_link">
@@ -35,6 +35,8 @@
     </joint>
     <gazebo reference="${name}_link">
-      <mu1>5.0</mu1>
-      <mu2>5.0</mu2>
+      <mu1>200.0</mu1>
+      <mu2>200.0</mu2>
+      <kp>1000000.0</kp>
+      <kd>100.0</kd>
       <material>Gazebo/Orange</material>
     </gazebo>

File: my_amr_description/urdf/gazebo_control.xacro (robot description, xacro)
@@ -15,5 +15,5 @@
       <frame_id>odom</frame_id>
       <child_frame_id>base_footprint</child_frame_id>
-      <publish_odom_tf>true</publish_odom_tf>
+      <publish_odom_tf>false</publish_odom_tf>
       <odom_publish_frequency>50</odom_publish_frequency>
     </plugin>

File: my_amr_description/urdf/robot_base.xacro (robot description, xacro)
@@ -5,5 +5,5 @@
   <xacro:property name="chassis_width"        value="0.40"/>
   <xacro:property name="chassis_height"       value="0.19"/>
-  <xacro:property name="chassis_mass"         value="12.0"/>
+  <xacro:property name="chassis_mass"         value="25.0"/>
   <xacro:property name="traction_wheel_radius" value="0.10"/>
   <xacro:property name="trolley_wheel_radius"  value="0.044"/>
@@ -82,4 +82,6 @@
       <mu1>0.0</mu1>
       <mu2>0.0</mu2>
+      <kp>1000000.0</kp>
+      <kd>100.0</kd>
       <material>Gazebo/Black</material>
     </gazebo>
