Commit message: feat(bcr_bot): tune navigation, lift, and mission executive for pick-and-place reliability
- Add pick_equivalent_yaw to allow front/back orientation flexibility for diff-drive bot
- Replace storage_approach waypoint with pickup_escape; switch footprint/inflation
  only after clearing pickup pillars to avoid costmap collision conflicts
- Remove PreferForwardCritic to allow reverse motion when goal is behind robot
- Reduce MPPI batch_size/time_steps and adjust vx_max for WSL2 performance
- Increase velocity deadband thresholds and loosen xy_goal_tolerance to fix
  goal-area oscillation
- Fix lift_joint upper limit (0.35 -> 0.4) to match commanded lift target
- Increase lift p_gain/i_gain/cmd_max to overcome assembly weight and joint friction
- Remove redundant/dead code (retreat_from_storage, unused scan_min_height handling)

File: urdf/lift.xacro (robot description, xacro)
@@ -33,5 +33,5 @@
             <origin xyz="0 0 0.18" rpy="0 0 0" />
             <axis xyz="0 0 1"/>
-            <limit lower="0.0" upper="0.35" effort="200.0" velocity="0.1"/>
+            <limit lower="0.0" upper="0.4" effort="200.0" velocity="0.3"/>
             <dynamics damping="10.0" friction="10.0"/>
         </joint>
@@ -49,11 +49,11 @@
                 <!-- Custom ROS 2 compatible topic name (no numbers as tokens!) -->
                 <topic>/bcr_bot/lift_joint/cmd_pos</topic>
-                <p_gain>500</p_gain>
-                <i_gain>10</i_gain>
-                <d_gain>50</d_gain>
-                <i_max>100</i_max>
-                <i_min>-100</i_min>
-                <cmd_max>200</cmd_max>
-                <cmd_min>-200</cmd_min>
+                <p_gain>1500</p_gain>
+                <i_gain>100</i_gain>
+                <d_gain>100</d_gain>
+                <i_max>300</i_max>
+                <i_min>-300</i_min>
+                <cmd_max>400</cmd_max>
+                <cmd_min>-400</cmd_min>
             </plugin>
         </gazebo>
